Commit message: new gluon_arm_bringup package created.

File: src/gluon_arm_description/urdf/gluon_ros2_control.xacro (robot description, xacro)
@@ -1,5 +1,5 @@
 <?xml version="1.0"?>
 <robot xmlns:xacro="http://www.ros.org/wiki/xacro" name="gluon">
-  <xacro:macro name="gluon_ros2_control" params="name">
+  <xacro:macro name="arm_controller" params="name">
     <ros2_control name="${name}" type="system">
       <hardware>
